File: kicad/80bus.kicad_pcb (KiCad board)
At the start: 2 copper layers, 203.2 x 203.2 mm, 119 parts, among them J1 Conn_01x80NasBus, P4 TestPoint, P5 TestPoint, P8 TestPoint, P9 TestPoint, SW1 SW_DIP_x08, U1 74LS245, U10 74LS32, U11 74LS02, U12 74LS195, U13 74LS273, U14 WD1793, U15 4013B, U16 7407, U17 74LS04, U18 74LS123, U19 7438, U2 74LS138, U20 4046B, U21 4016, U22 74LS14, U23 7406, U24 74LS123, U3 74LS10, U4 74LS04, U5 74LS365, U6 74LS163, U7 74LS257, U8 74LS257, U9 74LS32

Commit message: kicad8
Other:
- board text added: "4691c9db-ce99-49ee-8a38-c6e0fdd038de"
- board text added: "Errata -Update to KiCad 8"
- board text added: "Version 2.1.0"
- board text removed: "Errata -Update to KiCad 7"
- board text removed: "Version 2.0.0"
- board text removed: "fe52921d-bb14-464a-a215-66f4b561ce90"

Commit message: Document update / Kikad 9
Other:
- board text added: "3450fd75-a37b-4dd7-9636-6f1b02a52b20"
- board text added: "Errata -Update to KiCad 9"
- board text added: "Version 2.2.0"
- board text removed: "4691c9db-ce99-49ee-8a38-c6e0fdd038de"
- board text removed: "Errata -Update to KiCad 8"
- board text removed: "Version 2.1.0"

Commit message: Version update
Other:
- board text added: "CS-001"
Changed lines of the file:
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@@
 	(title_block
 		(title "Nascom FDC ")
-		(date "2025-03-30")
+		(date "2025-04-06")
 		(rev "2.2.0")
 		(comment 1 "Update to KiCad 9")
@@
 		)
 	)
+	(gr_text "CS-001"
+		(at 102.377824 229.7053 0)
+		(layer "B.SilkS")
+		(effects
+			(font
+				(size 1 1)
+				(thickness 0.15)
+			)
+			(justify left bottom mirror)
+		)
+	)

Commit message: Update docs
Parts:
- added G001: LOGO, 80bus:qr-code, B.Cu at (103.9, 77.3)
Other:
- board text added: "2b10c5f1-cc3f-4c91-b606-8f8e547184d4"
- board text added: "Docs -->"
- board text added: "Version 2.2.1"
- board text removed: "3450fd75-a37b-4dd7-9636-6f1b02a52b20"
- board text removed: "Version 2.2.0"
