File: kicad/address.kicad_sch (KiCad schematic)
At the start: 9 parts, among them SW1 SW_DIP_x08, U10 74LS32, U16 7407, U17 74LS04, U2 74LS138, U23 7406, U3 74LS10, U9 74LS32

Commit message: Document update / Kikad 9
Changed lines of the file:
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@@
 (kicad_sch
-	(version 20231120)
+	(version 20250114)
 	(generator "eeschema")
-	(generator_version "8.0")
+	(generator_version "9.0")
 	(paper "A3")
 	(title_block
 		(title "80 Bus FDC Controller")
-		(date "2025-02-09")
-		(rev "2.1.0")
+		(date "2025-03-30")
+		(rev "2.2.0")
+		(comment 1 "Update to Kicad 9")
 	)
 	(junction
@@
 			)
 		)
-		(property "Description" ""
+		(property "Description" "Hex Buffers and Drivers With Open Collector High Voltage Outputs"
 			(at 147.32 160.02 0)
 			(effects
@@
 			)
 		)
-		(property "Description" ""
+		(property "Description" "Power symbol creates a global label with name \"VCC\""
 			(at 172.72 83.82 0)
 			(effects
@@
 			)
 		)
-		(property "Description" ""
+		(property "Description" "Quad 2-input OR"
 			(at 292.1 127 0)
 			(effects
@@
 			)
 		)
-		(property "Description" ""
+		(property "Description" "Hex Inverter"
 			(at 147.32 114.3 0)
 			(effects
@@
 			)
 		)
-		(property "Description" ""
+		(property "Description" "Decoder 3 to 8 active low outputs"
 			(at 124.46 175.26 0)
 			(effects
@@
 			)
 		)
-		(property "Description" ""
+		(property "Description" "8x DIP Switch, Single Pole Single Throw (SPST) switch, small symbol"
 			(at 167.64 177.8 0)
 			(effects
@@
 			)
 		)
-		(property "Description" ""
+		(property "Description" "Quad 2-input OR"
 			(at 251.46 127 0)
 			(effects
@@
 			)
 		)
-		(property "Description" ""
+		(property "Description" "Triple 3-input NAND"
 			(at 304.8 167.64 0)
 			(effects
@@
 			)
 		)
-		(property "Description" ""
+		(property "Description" "Quad 2-input OR"
 			(at 193.04 208.28 0)
 			(effects
@@
 			)
 		)
-		(property "Description" ""
+		(property "Description" "Quad 2-input OR"
 			(at 266.7 144.78 0)
 			(effects
@@
 			)
 		)
-		(property "Description" ""
+		(property "Description" "Quad 2-input OR"
 			(at 266.7 180.34 0)
 			(effects
@@
 			)
 		)
-		(property "Description" ""
+		(property "Description" "Hex Inverter"
 			(at 236.22 165.1 0)
 			(effects
@@
 			)
 		)
-		(property "Description" ""
+		(property "Description" "Power symbol creates a global label with name \"VCC\""
 			(at 124.46 160.02 0)
 			(effects
@@
 			)
 		)
-		(property "Description" ""
+		(property "Description" "Hex Inverter"
 			(at 127 99.06 0)
 			(effects
@@
 			)
 		)
-		(property "Description" ""
+		(property "Description" "Inverter Open Collect"
 			(at 302.26 76.2 0)
 			(effects
@@
 			)
 		)
-		(property "Description" ""
+		(property "Description" "Hex Inverter"
 			(at 127 114.3 0)
 			(effects
@@
 			)
 		)
-		(property "Description" ""
+		(property "Description" "Quad 2-input OR"
 			(at 210.82 200.66 0)
 			(effects
@@
 			)
 		)
-		(property "Description" ""
+		(property "Description" "Quad 2-input OR"
 			(at 266.7 124.46 0)
 			(effects
@@
 			)
 		)
-		(property "Description" ""
+		(property "Description" "Resistor"
 			(at 163.83 83.82 0)
 			(effects
@@
 			)
 		)
-		(property "Description" ""
+		(property "Description" "Power symbol creates a global label with name \"GND\" , ground"
 			(at 124.46 193.04 0)
 			(effects
@@
 			)
 		)
-		(property "Description" ""
+		(property "Description" "Hex Inverter"
 			(at 147.32 129.54 0)
 			(effects
@@
 			)
 		)
-		(property "Description" ""
+		(property "Description" "Hex Inverter"
 			(at 147.32 99.06 0)
 			(effects
@@
 			)
 		)
-		(property "Description" ""
+		(property "Description" "Quad 2-input OR"
 			(at 210.82 215.9 0)
 			(effects
