File: kicad/data.kicad_sch (KiCad schematic)
At the start: 30 parts, among them P4 TestPoint, U1 74LS245, U13 74LS273, U18 74LS123, U3 74LS10, U4 74LS04, U5 74LS365, U6 74LS163, U7 74LS257, U8 74LS257

Commit message: Document update / Kikad 9
Changed lines of the file:
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@@
 (kicad_sch
-	(version 20231120)
+	(version 20250114)
 	(generator "eeschema")
-	(generator_version "8.0")
+	(generator_version "9.0")
 	(paper "A3")
 	(title_block
 		(title "80 Bus FDC Controller")
-		(date "2025-02-09")
-		(rev "2.1.0")
+		(date "2025-03-30")
+		(rev "2.2.0")
+		(comment 1 "Update to Kicad 9")
 	)
 	(junction
@@
 			)
 		)
-		(property "Description" ""
+		(property "Description" "Hex Inverter"
 			(at 261.62 187.96 0)
 			(effects
@@
 			)
 		)
-		(property "Description" ""
+		(property "Description" "Power symbol creates a global label with name \"GND\" , ground"
 			(at 284.48 132.08 0)
 			(effects
@@
 			)
 		)
-		(property "Description" ""
+		(property "Description" "Hex Bus Driver, 3-State Outputs"
 			(at 58.42 88.9 0)
 			(effects
@@
 			)
 		)
-		(property "Description" ""
+		(property "Description" "Power symbol creates a global label with name \"GND\" , ground"
 			(at 236.22 81.28 0)
 			(effects
@@
 			)
 		)
-		(property "Description" ""
+		(property "Description" "Power symbol creates a global label with name \"GND\" , ground"
 			(at 58.42 187.96 0)
 			(effects
@@
 			)
 		)
-		(property "Description" ""
+		(property "Description" "Power symbol creates a global label with name \"VCC\""
 			(at 43.18 121.92 0)
 			(effects
@@
 			)
 		)
-		(property "Description" ""
+		(property "Description" "Power symbol creates a global label with name \"VCC\""
 			(at 27.94 121.92 0)
 			(effects
@@
 			)
 		)
-		(property "Description" ""
+		(property "Description" "Jumper, 2-pole, open"
 			(at 134.62 228.6 0)
 			(effects
@@
 			)
 		)
-		(property "Description" ""
+		(property "Description" "Power symbol creates a global label with name \"VCC\""
 			(at 127 210.82 0)
 			(effects
@@
 			)
 		)
-		(property "Description" ""
+		(property "Description" "Synchronous 4-bit programmable binary Counter"
 			(at 294.64 198.12 0)
 			(effects
@@
 			)
 		)
-		(property "Description" ""
+		(property "Description" "Hex Inverter"
 			(at 58.42 254 0)
 			(effects
@@
 			)
 		)
-		(property "Description" ""
+		(property "Description" "Dual retriggerable Monostable"
 			(at 312.42 134.62 0)
 			(effects
@@
 			)
 		)
-		(property "Description" ""
+		(property "Description" "Resistor"
 			(at 323.85 149.86 0)
 			(effects
@@
 			)
 		)
-		(property "Description" ""
+		(property "Description" "Hex Inverter"
 			(at 337.82 38.1 0)
 			(effects
@@
 			)
 		)
-		(property "Description" ""
+		(property "Description" "Power symbol creates a global label with name \"GND\" , ground"
 			(at 154.94 71.12 0)
 			(effects
@@
 			)
 		)
-		(property "Description" ""
+		(property "Description" "Resistor"
 			(at 224.79 269.24 0)
 			(effects
@@
 			)
 		)
-		(property "Description" ""
+		(property "Description" "Power symbol creates a global label with name \"GND\" , ground"
 			(at 58.42 106.68 0)
 			(effects
@@
 			)
 		)
-		(property "Description" ""
+		(property "Description" "Power symbol creates a global label with name \"VCC\""
 			(at 353.06 119.38 0)
 			(effects
@@
 			)
 		)
-		(property "Description" ""
+		(property "Description" "Polarized capacitor"
 			(at 240.03 93.98 0)
 			(effects
@@
 			)
 		)
-		(property "Description" ""
+		(property "Description" "Resistor"
 			(at 323.85 236.22 0)
 			(effects
@@
 			)
 		)
-		(property "Description" ""
+		(property "Description" "Resistor"
 			(at 35.56 118.11 0)
 			(effects
@@
 			)
 		)
-		(property "Description" ""
+		(property "Description" "Resistor"
 			(at 43.18 118.11 0)
 			(effects
@@
 			)
 		)
-		(property "Description" ""
+		(property "Description" "Quad 2 to 1 Multiplexer"
 			(at 134.62 43.18 0)
 			(effects
@@
 			)
 		)
-		(property "Description" ""
+		(property "Description" "Power symbol creates a global label with name \"VCC\""
 			(at 246.38 81.28 0)
 			(effects
@@
 			)
 		)
-		(property "Description" ""
+		(property "Description" "test point"
 			(at 332.74 233.68 0)
 			(effects
@@
 			)
 		)
-		(property "Description" ""
+		(property "Description" "Resistor"
 			(at 346.71 119.38 0)
 			(effects
@@
 			)
 		)
-		(property "Description" ""
+		(property "Description" "Power symbol creates a global label with name \"VCC\""
 			(at 297.18 111.76 0)
 			(effects
@@
 			)
 		)
-		(property "Description" ""
+		(property "Description" "Power symbol creates a global label with name \"VCC\""
 			(at 185.42 96.52 0)
 			(effects
@@
 			)
 		)
-		(property "Description" ""
+		(property "Description" "Resistor"
 			(at 297.18 115.57 0)
 			(effects
@@
 			)
 		)
-		(property "Description" ""
+		(property "Description" "Dual retriggerable Monostable"
 			(at 261.62 109.22 0)
 			(effects
@@
 			)
 		)
-		(property "Description" ""
+		(property "Description" "Power symbol creates a global label with name \"VCC\""
 			(at 58.42 147.32 0)
 			(effects
@@
 			)
 		)
-		(property "Description" ""
+		(property "Description" "Power symbol creates a global label with name \"VCC\""
 			(at 58.42 71.12 0)
 			(effects
@@
 			)
 		)
-		(property "Description" ""
+		(property "Description" "Resistor"
 			(at 123.19 226.06 0)
 			(effects
@@
 			)
 		)
-		(property "Description" ""
+		(property "Description" "Resistor"
 			(at 283.21 22.86 0)
 			(effects
@@
 			)
 		)
-		(property "Description" ""
+		(property "Description" "Resistor"
 			(at 123.19 210.82 0)
 			(effects
@@
 			)
 		)
-		(property "Description" ""
+		(property "Description" "Hex Inverter"
 			(at 264.16 210.82 0)
 			(effects
@@
 			)
 		)
-		(property "Description" ""
+		(property "Description" "Power symbol creates a global label with name \"VCC\""
 			(at 320.04 236.22 0)
 			(effects
@@
 			)
 		)
-		(property "Description" ""
+		(property "Description" "test point"
 			(at 200.66 121.92 0)
 			(effects
@@
 			)
 		)
-		(property "Description" ""
+		(property "Description" "Power symbol creates a global label with name \"VCC\""
 			(at 127 226.06 0)
 			(effects
@@
 			)
 		)
-		(property "Description" ""
+		(property "Description" "Quad 2 to 1 Multiplexer"
 			(at 99.06 220.98 0)
 			(effects
@@
 			)
 		)
-		(property "Description" ""
+		(property "Description" "Generic connector, double row, 02x10, counter clockwise pin numbering scheme (similar to DIP package numbering), script generated (kicad-library-utils/schlib/autogen/connector/)"
 			(at 266.7 231.14 0)
 			(effects
@@
 			)
 		)
-		(property "Description" ""
+		(property "Description" "Power symbol creates a global label with name \"VCC\""
 			(at 246.38 241.3 0)
 			(effects
@@
 			)
 		)
-		(property "Description" ""
+		(property "Description" "Polarized capacitor"
 			(at 290.83 121.92 0)
 			(effects
@@
 			)
 		)
-		(property "Description" ""
+		(property "Description" "Jumper, 2-pole, open"
 			(at 134.62 213.36 0)
 			(effects
@@
 			)
 		)
-		(property "Description" ""
+		(property "Description" "Power symbol creates a global label with name \"VCC\""
 			(at 134.62 20.32 0)
 			(effects
@@
 			)
 		)
-		(property "Description" ""
+		(property "Description" "Power symbol creates a global label with name \"VCC\""
 			(at 289.56 22.86 0)
 			(effects
@@
 			)
 		)
-		(property "Description" ""
+		(property "Description" "8-bit D Flip-Flop, reset"
 			(at 185.42 116.84 0)
 			(effects
@@
 			)
 		)
-		(property "Description" ""
+		(property "Description" "Power symbol creates a global label with name \"VCC\""
 			(at 314.96 198.12 0)
 			(effects
@@
 			)
 		)
-		(property "Description" ""
+		(property "Description" "Resistor"
 			(at 285.75 233.68 0)
 			(effects
@@
 			)
 		)
-		(property "Description" ""
+		(property "Description" "Power symbol creates a global label with name \"GND\" , ground"
 			(at 124.46 248.92 0)
 			(effects
@@
 			)
 		)
-		(property "Description" ""
+		(property "Description" "Power symbol creates a global label with name \"VCC\""
 			(at 99.06 198.12 0)
 			(effects
@@
 			)
 		)
-		(property "Description" ""
+		(property "Description" "Power symbol creates a global label with name \"VCC\""
 			(at 289.56 233.68 0)
 			(effects
@@
 			)
 		)
-		(property "Description" ""
+		(property "Description" "Power symbol creates a global label with name \"GND\" , ground"
 			(at 274.32 198.12 0)
 			(effects
@@
 			)
 		)
-		(property "Description" ""
+		(property "Description" "Power symbol creates a global label with name \"GND\" , ground"
 			(at 289.56 223.52 0)
 			(effects
@@
 			)
 		)
-		(property "Description" ""
+		(property "Description" "Power symbol creates a global label with name \"VCC\""
 			(at 330.2 149.86 0)
 			(effects
@@
 			)
 		)
-		(property "Description" ""
+		(property "Description" "Resistor"
 			(at 252.73 241.3 0)
 			(effects
@@
 			)
 		)
-		(property "Description" ""
+		(property "Description" "Power symbol creates a global label with name \"GND\" , ground"
 			(at 185.42 137.16 0)
 			(effects
@@
 			)
 		)
-		(property "Description" ""
+		(property "Description" "Resistor"
 			(at 246.38 85.09 0)
 			(effects
@@
 			)
 		)
-		(property "Description" ""
+		(property "Description" "Power symbol creates a global label with name \"VCC\""
 			(at 218.44 269.24 0)
 			(effects
@@
 			)
 		)
-		(property "Description" ""
+		(property "Description" "Power symbol creates a global label with name \"VCC\""
 			(at 35.56 121.92 0)
 			(effects
@@
 			)
 		)
-		(property "Description" ""
+		(property "Description" "Resistor"
 			(at 27.94 118.11 0)
 			(effects
@@
 			)
 		)
-		(property "Description" ""
+		(property "Description" "Octal BUS Transceivers, 3-State outputs"
 			(at 58.42 167.64 0)
 			(effects
@@
 			)
 		)
-		(property "Description" ""
+		(property "Description" "Triple 3-input NAND"
 			(at 337.82 106.68 0)
 			(effects
